File: Impedance_Board/Impedance.brd (EAGLE design)
At the start: 65 x 56 mm, 35 parts, among them J1 SJ-3523-SMT-TR, J3 I2C, J4 I2C, J6 SJ-3523-SMT-TR, J7 SJ-3523-SMT-TR, U1 ANALOG_DEVICES_AD5933YRSZANAL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, U2 INA826AID, U7 AD8606ARZ, U8 AD8606ARZ, X1 RASPI_BOARD_B+#_H

Commit message: Impedance Circuit Explanation
Routing:
- net N$5: track 9.14 -> 31.3 mm
- net GND: track 13.5 -> 22.8 mm, vias 2 -> 3
- net N$8: track 35.9 -> 35.2 mm
