File: ECG_Board/ECG 7 by 7.sch (EAGLE design)
At the start: 7 parts

Commit message: Cleanup, organization and updates
Parts:
- removed JP1: (no value), SparkFun-Connectors:M03PTH
- removed JP3: (no value), SparkFun-Connectors:M06SIP
- added FRAME1: FRAME-LETTERNO_PACKAGE, SparkFun-Aesthetics:FRAME-LETTERNO_PACKAGE
- added U$1: (no value), SPARK_ECG:SPARK_ECG
Connections:
- net 3.3V: now also U$1.3.3V; no longer JP3.2
- net GND: now also U$1.GND; no longer JP3.1
- net N$1: now also U$1.RA; no longer JP1.1
- net N$2: now also U$1.LA; no longer JP1.2
- net N$3: now also U$1.RL; no longer JP1.3
- net N$4: now also U$1.!SDN; no longer JP3.6
- net N$5: now also U$1.LO+; no longer JP3.5
- net N$6: now also U$1.LO-; no longer JP3.4
- net N$7: now also U$1.OUT; no longer JP3.3
Other:
- moved on the sheet: JP2, JP4
