File: Airquality/Airquality.sch (EAGLE design)
At the start: 67 parts, among them IC1 SCD41-D-R2, U1 SGP41-D-R4, U3 BMP581, U4 AP22802AW5-7K-3.3V

Commit message: Air Quality at 3.3V with 5V boost for PM sensor
Parts:
- removed JP4: JUMPER-SMT_2_NO_SILK, SparkFun-Jumpers:JUMPER-SMT_2_NO_SILK
- added C17, C18, C19, C20, C21, C22, C23, C24: 0.1uF, SparkFun-Capacitors:0.1UF-0402-16V-10%
- added C25: 1.0uF, SparkFun-Capacitors:1.0UF-0402-16V-10%
- added C26, C27: 10uF, SparkFun-Capacitors:10UF-0603-6.3V-20%
- added U5: AP3602AKTR-G1, AP3602A:AP3602AKTR-G1
- C12, C13, C14, C15: value 10uF -> 0.1uF; device SparkFun-Capacitors:10UF-0603-6.3V-20% -> SparkFun-Capacitors:0.1UF-0402-16V-10%
- J4: device SparkFun-Connectors:CONN_07 -> SparkFun-Connectors:CONN_06SILK_FEMALE_PTH
- R10: value 130 -> 61; device SparkFun-Resistors:1.20KOHM-0603-1/10W-1% -> SparkFun-Resistors:82OHM-0603-1/10W-1%
- R3: value 10 -> 0
- R4: value 10 -> 4.7
- R8: value 820 -> 29; device SparkFun-Resistors:866OHM-0603-1/10W-1% -> SparkFun-Resistors:27OHM-0603-1/10W-1%
- R9: value 27 -> 38; device SparkFun-Resistors:20OHM-0603-1/10W-1% -> SparkFun-Resistors:33OHM-0603-1/10W-1%
Connections:
- removed net 5V: C12.1, C13.1, C14.1, C15.1, C7.1, J2.1, J4.1, J5.3, JP4.1, JP4.2, LED0.VDD, LED1.VDD, LED10.VDD, LED11.VDD, LED2.VDD, LED3.VDD, LED4.VDD, LED5.VDD, LED6.VDD, LED7.VDD, LED8.VDD, LED9.VDD, R7.1, U4.IN
- new net N$15: C25.1, U5.C+
- new net N$30: C25.2, U5.C-
- new net N$31: C12.1, C13.1, C14.1, C15.1, C17.1, C18.1, C19.1, C20.1, C21.1, C22.1, C23.1, C24.1, J5.3, LED0.VDD, LED1.VDD, LED10.VDD, LED11.VDD, LED2.VDD, LED3.VDD, LED4.VDD, LED5.VDD, LED6.VDD, LED7.VDD, LED8.VDD, LED9.VDD
- new net VOUT: C26.1, J2.1, U5.VOUT
- net 3.3V: now also C27.1, C7.1, J4.1, R7.1, U4.IN, U5.!SHDN, U5.VIN; no longer J4.7
- net GND: now also C17.2, C18.2, C19.2, C20.2, C21.2, C22.2, C23.2, C24.2, C26.2, C27.2, U2.E, U5.GND
- net N$13: no longer U2.E
Other:
- note added: "CO"
- note added: "NH3"
- note added: "NO2"
- moved on the sheet: C13, C14, C15

Commit message: BOM
Parts:
- added FLG: TEST-POINT3X4, SparkFun-Connectors:TEST-POINT3X4
- added R15: 10k, SparkFun-Resistors:10KOHM-0603-1/10W-1%
Connections:
- removed net N$9: J4.2, U4.EN
- new net N$32: J4.2, R15.2, U4.EN
- net 3.3V: now also R15.1
- net N$3: now also FLG.1
Changed lines of the file:
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@@
 <part name="SUPPLY7" library="SparkFun-PowerSymbols" library_urn="urn:adsk.eagle:library:530" deviceset="VOUT" device=""/>
 <part name="SUPPLY3" library="SparkFun-PowerSymbols" library_urn="urn:adsk.eagle:library:530" deviceset="VOUT" device=""/>
+<part name="R15" library="SparkFun-Resistors" library_urn="urn:adsk.eagle:library:532" deviceset="10KOHM" device="-0603-1/10W-1%" package3d_urn="urn:adsk.eagle:package:39650/1" value="10k"/>
+<part name="FLG" library="SparkFun-Connectors" library_urn="urn:adsk.eagle:library:513" deviceset="TEST-POINT" device="3X4" package3d_urn="urn:adsk.eagle:package:38287/1"/>
 </parts>
 <sheets>
@@
 <instance part="SUPPLY3" gate="G$1" x="-78.74" y="-48.26" smashed="yes">
 <attribute name="VALUE" x="-78.74" y="-45.466" size="1.778" layer="96" align="bottom-center"/>
+</instance>
+<instance part="R15" gate="G$1" x="25.4" y="58.42" smashed="yes">
+<attribute name="NAME" x="25.4" y="59.944" size="1.778" layer="95" font="vector" align="bottom-center"/>
+<attribute name="VALUE" x="25.4" y="56.896" size="1.778" layer="96" font="vector" align="top-center"/>
+</instance>
+<instance part="FLG" gate="G$1" x="30.48" y="76.2" smashed="yes" rot="R90">
+<attribute name="NAME" x="25.4" y="76.2" size="1.778" layer="95" font="vector"/>
+<attribute name="VALUE" x="33.02" y="73.66" size="1.778" layer="96" font="vector" rot="R90" display="off"/>
 </instance>
 </instances>
@@
 <wire x1="20.32" y1="76.2" x2="20.32" y2="71.12" width="0.1524" layer="91"/>
 <pinref part="SUPPLY4" gate="G$1" pin="3.3V"/>
+<pinref part="R15" gate="G$1" pin="1"/>
+<wire x1="20.32" y1="66.04" x2="20.32" y2="58.42" width="0.1524" layer="91"/>
+<junction x="20.32" y="66.04"/>
 </segment>
 <segment>
@@
 </segment>
 </net>
-<net name="N$9" class="0">
-<segment>
-<pinref part="U4" gate="G$1" pin="EN"/>
-<wire x1="20.32" y1="-2.54" x2="20.32" y2="60.96" width="0.1524" layer="91"/>
-<wire x1="33.02" y1="60.96" x2="20.32" y2="60.96" width="0.1524" layer="91"/>
-<pinref part="J4" gate="G$1" pin="2"/>
-<wire x1="15.24" y1="-2.54" x2="20.32" y2="-2.54" width="0.1524" layer="91"/>
-</segment>
-</net>
 <net name="N$13" class="0">
 <segment>
@@
 <pinref part="U4" gate="G$1" pin="FLG"/>
 <wire x1="30.48" y1="66.04" x2="33.02" y2="66.04" width="0.1524" layer="91"/>
+<wire x1="30.48" y1="66.04" x2="30.48" y2="76.2" width="0.1524" layer="91"/>
+<junction x="30.48" y="66.04"/>
+<pinref part="FLG" gate="G$1" pin="1"/>
 </segment>
 </net>
@@
 </segment>
 </net>
+<net name="N$32" class="0">
+<segment>
+<pinref part="R15" gate="G$1" pin="2"/>
+<wire x1="30.48" y1="58.42" x2="30.48" y2="60.96" width="0.1524" layer="91"/>
+<pinref part="U4" gate="G$1" pin="EN"/>
+<wire x1="30.48" y1="60.96" x2="33.02" y2="60.96" width="0.1524" layer="91"/>
+<wire x1="30.48" y1="58.42" x2="30.48" y2="53.34" width="0.1524" layer="91"/>
+<junction x="30.48" y="58.42"/>
+<wire x1="30.48" y1="53.34" x2="20.32" y2="53.34" width="0.1524" layer="91"/>
+<pinref part="J4" gate="G$1" pin="2"/>
+<wire x1="15.24" y1="-2.54" x2="20.32" y2="-2.54" width="0.1524" layer="91"/>
+<wire x1="20.32" y1="53.34" x2="20.32" y2="-2.54" width="0.1524" layer="91"/>
+</segment>
+</net>

Commit message: Production Updates
Parts:
- U5: device AP3602A:AP3602AKTR-G1 -> AP3602AKTR-G1:AP3602AKTR-G1
Other:
- moved on the sheet: C26
Changed lines of the file:
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@@
 <drawing>
 <settings>
-<setting alwaysvectorfont="no"/>
+<setting alwaysvectorfont="yes"/>
 <setting verticaltext="up"/>
 </settings>
@@
 <part name="C13" library="SparkFun-Capacitors" library_urn="urn:adsk.eagle:library:510" deviceset="0.1UF" device="-0402-16V-10%" package3d_urn="urn:adsk.eagle:package:37413/1" value="0.1uF"/>
 <part name="C24" library="SparkFun-Capacitors" library_urn="urn:adsk.eagle:library:510" deviceset="0.1UF" device="-0402-16V-10%" package3d_urn="urn:adsk.eagle:package:37413/1" value="0.1uF"/>
-<part name="U5" library="AP3602A" deviceset="AP3602AKTR-G1" device=""/>
+<part name="U5" library="AP3602AKTR-G1" deviceset="AP3602AKTR-G1" device=""/>
 <part name="SUPPLY4" library="SparkFun-PowerSymbols" library_urn="urn:adsk.eagle:library:530" deviceset="3.3V" device=""/>
 <part name="SUPPLY6" library="SparkFun-PowerSymbols" library_urn="urn:adsk.eagle:library:530" deviceset="3.3V" device=""/>
@@
 <attribute name="VALUE" x="116.586" y="-14.859" size="1.778" layer="96" font="vector"/>
 </instance>
-<instance part="U5" gate="A" x="81.28" y="73.66" smashed="yes">
+<instance part="U5" gate="G$1" x="81.28" y="73.66" smashed="yes">
 <attribute name="NAME" x="91.5416" y="76.4286" size="2.0828" layer="95" ratio="20" rot="SR0"/>
-<attribute name="VALUE" x="91.6686" y="63.5254" size="2.0828" layer="96" ratio="10" rot="SR0"/>
+<attribute name="VALUE" x="86.5886" y="63.5254" size="2.0828" layer="96" ratio="10" rot="SR0"/>
 </instance>
 <instance part="SUPPLY4" gate="G$1" x="20.32" y="76.2" smashed="yes">
@@
 <attribute name="VALUE" x="118.364" y="68.961" size="1.778" layer="96" font="vector"/>
 </instance>
-<instance part="C26" gate="G$1" x="78.74" y="68.58" smashed="yes">
-<attribute name="NAME" x="80.264" y="71.501" size="1.778" layer="95" font="vector"/>
-<attribute name="VALUE" x="80.264" y="66.421" size="1.778" layer="96" font="vector"/>
+<instance part="C26" gate="G$1" x="76.2" y="68.58" smashed="yes">
+<attribute name="NAME" x="77.724" y="71.501" size="1.778" layer="95" font="vector"/>
+<attribute name="VALUE" x="77.724" y="66.421" size="1.778" layer="96" font="vector"/>
 </instance>
 <instance part="C27" gate="G$1" x="111.76" y="60.96" smashed="yes">
@@
 <attribute name="VALUE" x="111.76" y="55.626" size="1.778" layer="96" align="top-center"/>
 </instance>
-<instance part="GND20" gate="1" x="81.28" y="63.5" smashed="yes">
-<attribute name="VALUE" x="81.28" y="63.246" size="1.778" layer="96" align="top-center"/>
-</instance>
-<instance part="SUPPLY7" gate="G$1" x="78.74" y="76.2" smashed="yes">
-<attribute name="VALUE" x="78.74" y="78.994" size="1.778" layer="96" align="bottom-center"/>
+<instance part="GND20" gate="1" x="78.74" y="63.5" smashed="yes">
+<attribute name="VALUE" x="78.74" y="62.992" size="1.778" layer="96" align="top-center"/>
+</instance>
+<instance part="SUPPLY7" gate="G$1" x="76.2" y="76.2" smashed="yes">
+<attribute name="VALUE" x="76.2" y="78.994" size="1.778" layer="96" align="bottom-center"/>
 </instance>
 <instance part="SUPPLY3" gate="G$1" x="-78.74" y="-48.26" smashed="yes">
@@
 <pinref part="C26" gate="G$1" pin="2"/>
 <pinref part="GND20" gate="1" pin="GND"/>
-<pinref part="U5" gate="A" pin="GND"/>
-<wire x1="88.9" y1="71.12" x2="83.82" y2="71.12" width="0.1524" layer="91"/>
-<wire x1="83.82" y1="71.12" x2="83.82" y2="66.04" width="0.1524" layer="91"/>
-<wire x1="83.82" y1="66.04" x2="78.74" y2="66.04" width="0.1524" layer="91"/>
+<pinref part="U5" gate="G$1" pin="GND"/>
+<wire x1="81.28" y1="71.12" x2="78.74" y2="71.12" width="0.1524" layer="91"/>
+<wire x1="78.74" y1="71.12" x2="78.74" y2="66.04" width="0.1524" layer="91"/>
 <junction x="78.74" y="66.04"/>
-<wire x1="78.74" y1="66.04" x2="81.28" y2="66.04" width="0.1524" layer="91"/>
+<wire x1="76.2" y1="66.04" x2="78.74" y2="66.04" width="0.1524" layer="91"/>
 </segment>
 </net>
@@
 </segment>
 <segment>
-<pinref part="U5" gate="A" pin="VIN"/>
+<pinref part="U5" gate="G$1" pin="VIN"/>
 <wire x1="109.22" y1="71.12" x2="111.76" y2="71.12" width="0.1524" layer="91"/>
 <pinref part="C27" gate="G$1" pin="1"/>
@@
 <junction x="111.76" y="71.12"/>
 <pinref part="SUPPLY2" gate="G$1" pin="3.3V"/>
-<pinref part="U5" gate="A" pin="!SHDN"/>
-<wire x1="88.9" y1="68.58" x2="86.36" y2="68.58" width="0.1524" layer="91"/>
-<wire x1="86.36" y1="68.58" x2="86.36" y2="78.74" width="0.1524" layer="91"/>
-<wire x1="86.36" y1="78.74" x2="111.76" y2="78.74" width="0.1524" layer="91"/>
+<pinref part="U5" gate="G$1" pin="!SHDN"/>
+<wire x1="81.28" y1="68.58" x2="80.01" y2="68.58" width="0.1524" layer="91"/>
+<wire x1="80.01" y1="68.58" x2="80.01" y2="78.74" width="0.1524" layer="91"/>
+<wire x1="80.01" y1="78.74" x2="111.76" y2="78.74" width="0.1524" layer="91"/>
 <junction x="111.76" y="78.74"/>
 </segment>
@@
 <net name="N$15" class="0">
 <segment>
-<pinref part="U5" gate="A" pin="C+"/>
+<pinref part="U5" gate="G$1" pin="C+"/>
 <wire x1="109.22" y1="73.66" x2="114.3" y2="73.66" width="0.1524" layer="91"/>
 <pinref part="C25" gate="G$1" pin="1"/>
@@
 <segment>
 <pinref part="C25" gate="G$1" pin="2"/>
-<pinref part="U5" gate="A" pin="C-"/>
+<pinref part="U5" gate="G$1" pin="C-"/>
 <wire x1="116.84" y1="68.58" x2="109.22" y2="68.58" width="0.1524" layer="91"/>
 </segment>
@@
 </segment>
 <segment>
-<pinref part="U5" gate="A" pin="VOUT"/>
+<pinref part="U5" gate="G$1" pin="VOUT"/>
 <pinref part="C26" gate="G$1" pin="1"/>
-<wire x1="88.9" y1="73.66" x2="78.74" y2="73.66" width="0.1524" layer="91"/>
+<wire x1="81.28" y1="73.66" x2="76.2" y2="73.66" width="0.1524" layer="91"/>
 <pinref part="SUPPLY7" gate="G$1" pin="VOUT"/>
-<wire x1="78.74" y1="73.66" x2="78.74" y2="76.2" width="0.1524" layer="91"/>
-<junction x="78.74" y="73.66"/>
-</segment>
-</net>
+<wire x1="76.2" y1="73.66" x2="76.2" y2="76.2" width="0.1524" layer="91"/>
+<junction x="76.2" y="73.66"/>
+</segment>
+</net>
