File: Impedance_Potential_Board/Impedance_Potential.sch (EAGLE design)
At the start: 85 parts, among them IC1 MAX30001GCWV+, J1 Header, U4 AP2112K-1.8V

Commit message: Production Updates
Parts:
- U4: device SparkFun-PowerIC:V_REG_LDOSMD -> AP2112K-1.8TRG1:AP2122K-1.8TRG1SMD
- renumbered EC_UNBAL to EC_UB, EN_UNBAL to EN_UB, EP_UNBAL to EP_UB
Changed lines of the file:
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@@
 <drawing>
 <settings>
-<setting alwaysvectorfont="no"/>
+<setting alwaysvectorfont="yes"/>
 <setting verticaltext="up"/>
 </settings>
-<grid distance="0.1" unitdist="inch" unit="inch" style="lines" multiple="1" display="yes" altdistance="0.01" altunitdist="inch" altunit="inch"/>
+<grid distance="0.1" unitdist="inch" unit="inch" style="lines" multiple="1" display="no" altdistance="0.01" altunitdist="inch" altunit="inch"/>
 <layers>
 <layer number="1" name="Top" color="4" fill="1" visible="no" active="no"/>
+<layer number="2" name="Route2" color="1" fill="3" visible="no" active="no"/>
+<layer number="3" name="Route3" color="4" fill="3" visible="no" active="no"/>
+<layer number="4" name="Route4" color="1" fill="4" visible="no" active="no"/>
+<layer number="5" name="Route5" color="4" fill="4" visible="no" active="no"/>
+<layer number="6" name="Route6" color="1" fill="8" visible="no" active="no"/>
+<layer number="7" name="Route7" color="4" fill="8" visible="no" active="no"/>
+<layer number="8" name="Route8" color="1" fill="2" visible="no" active="no"/>
+<layer number="9" name="Route9" color="4" fill="2" visible="no" active="no"/>
+<layer number="10" name="Route10" color="1" fill="7" visible="no" active="no"/>
+<layer number="11" name="Route11" color="4" fill="7" visible="no" active="no"/>
+<layer number="12" name="Route12" color="1" fill="5" visible="no" active="no"/>
+<layer number="13" name="Route13" color="4" fill="5" visible="no" active="no"/>
+<layer number="14" name="Route14" color="1" fill="6" visible="no" active="no"/>
+<layer number="15" name="Route15" color="4" fill="6" visible="no" active="no"/>
 <layer number="16" name="Bottom" color="1" fill="1" visible="no" active="no"/>
 <layer number="17" name="Pads" color="2" fill="1" visible="no" active="no"/>
@@
 <part name="GND4" library="SparkFun-Aesthetics" deviceset="GND" device=""/>
 <part name="LED_ENABLE" library="SparkFun-Jumpers" library_urn="urn:adsk.eagle:library:528" deviceset="JUMPER-SMT_2_NC_PASTE" device="_SILK" package3d_urn="urn:adsk.eagle:package:39282/1" value="LED ENABLE"/>
-<part name="FRAME1" library="SparkFun-Aesthetics" library_urn="urn:adsk.eagle:library:507" deviceset="FRAME-LETTER" device="NO_PACKAGE" package3d_urn="urn:adsk.eagle:package:37104/1"/>
+<part name="FRAME1" library="SparkFun-Aesthetics" library_urn="urn:adsk.eagle:library:507" deviceset="FRAME-LETTER" device="NO_PACKAGE" package3d_urn="urn:adsk.eagle:package:41384587/3"/>
 <part name="IC1" library="MAX30001GCWV+" deviceset="MAX30001GCWV+" device=""/>
 <part name="C1" library="SparkFun-Capacitors" library_urn="urn:adsk.eagle:library:510" deviceset="0.22UF" device="-0603-25V-10%" package3d_urn="urn:adsk.eagle:package:37414/1" value="0.22uF"/>
@@
 <part name="C16" library="SparkFun-Capacitors" deviceset="1.0UF" device="-0603-16V-10%" value="1.0uF"/>
 <part name="GND35" library="supply1" deviceset="GND" device=""/>
-<part name="U4" library="SparkFun-PowerIC" deviceset="V_REG_LDO" device="SMD" value="AP2112K-1.8V">
+<part name="U4" library="AP2112K-1.8TRG1" deviceset="AP2122K-1.8TRG1" device="SMD" value="AP2112K-1.8V">
 <attribute name="PROD_ID" value="VREG-12457"/>
 </part>
@@
 <part name="SUPPLY15" library="SparkFun-PowerSymbols" library_urn="urn:adsk.eagle:library:530" deviceset="3.3V" device=""/>
 <part name="SUPPLY16" library="SparkFun-PowerSymbols" library_urn="urn:adsk.eagle:library:530" deviceset="3.3V" device=""/>
-<part name="EP_UNBAL" library="SparkFun-Jumpers" library_urn="urn:adsk.eagle:library:528" deviceset="JUMPER-SMT_2_NO" device="_SILK" package3d_urn="urn:adsk.eagle:package:39279/1" value="JUMPER-SMT_2_NO_SILK"/>
-<part name="EN_UNBAL" library="SparkFun-Jumpers" library_urn="urn:adsk.eagle:library:528" deviceset="JUMPER-SMT_2_NO" device="_SILK" package3d_urn="urn:adsk.eagle:package:39279/1" value="JUMPER-SMT_2_NO_SILK"/>
+<part name="EP_UB" library="SparkFun-Jumpers" library_urn="urn:adsk.eagle:library:528" deviceset="JUMPER-SMT_2_NO" device="_SILK" package3d_urn="urn:adsk.eagle:package:39279/1" value="JUMPER-SMT_2_NO_SILK"/>
+<part name="EN_UB" library="SparkFun-Jumpers" library_urn="urn:adsk.eagle:library:528" deviceset="JUMPER-SMT_2_NO" device="_SILK" package3d_urn="urn:adsk.eagle:package:39279/1" value="JUMPER-SMT_2_NO_SILK"/>
 <part name="C24" library="SparkFun-Capacitors" library_urn="urn:adsk.eagle:library:510" deviceset="47NF" device="-0603-25V-5%" package3d_urn="urn:adsk.eagle:package:37414/1" value="47nF"/>
-<part name="EC_UNBAL" library="SparkFun-Jumpers" library_urn="urn:adsk.eagle:library:528" deviceset="JUMPER-SMT_2_NO" device="_SILK" package3d_urn="urn:adsk.eagle:package:39279/1" value="JUMPER-SMT_2_NO_SILK"/>
+<part name="EC_UB" library="SparkFun-Jumpers" library_urn="urn:adsk.eagle:library:528" deviceset="JUMPER-SMT_2_NO" device="_SILK" package3d_urn="urn:adsk.eagle:package:39279/1" value="JUMPER-SMT_2_NO_SILK"/>
 <part name="SUPPLY19" library="SparkFun-PowerSymbols" library_urn="urn:adsk.eagle:library:530" deviceset="3.3V" device=""/>
 <part name="R19" library="SparkFun-Resistors" library_urn="urn:adsk.eagle:library:532" deviceset="0OHM" device="-0603-1/10W-5%" package3d_urn="urn:adsk.eagle:package:39650/1" value="0"/>
@@
 <attribute name="VALUE" x="-120.65" y="35.814" size="1.778" layer="96" align="bottom-center"/>
 </instance>
-<instance part="EP_UNBAL" gate="G$1" x="76.2" y="-3.81" smashed="yes" rot="R90">
+<instance part="EP_UB" gate="G$1" x="76.2" y="-3.81" smashed="yes" rot="R90">
 <attribute name="NAME" x="79.248" y="-8.128" size="1.778" layer="95" font="vector" rot="R90"/>
 </instance>
-<instance part="EN_UNBAL" gate="G$1" x="67.31" y="-22.86" smashed="yes" rot="R90">
+<instance part="EN_UB" gate="G$1" x="67.31" y="-22.86" smashed="yes" rot="R90">
 <attribute name="NAME" x="70.612" y="-27.178" size="1.778" layer="95" font="vector" rot="R90"/>
 </instance>
@@
 <attribute name="VALUE" x="39.878" y="-27.051" size="1.778" layer="96" font="vector" rot="MR270"/>
 </instance>
-<instance part="EC_UNBAL" gate="G$1" x="48.26" y="-25.4" smashed="yes" rot="R90">
+<instance part="EC_UB" gate="G$1" x="48.26" y="-25.4" smashed="yes" rot="R90">
 <attribute name="NAME" x="51.562" y="-29.718" size="1.778" layer="95" font="vector" rot="R90"/>
 </instance>
@@
 <junction x="76.2" y="-8.89"/>
 <junction x="76.2" y="-8.89"/>
-<pinref part="EP_UNBAL" gate="G$1" pin="1"/>
+<pinref part="EP_UB" gate="G$1" pin="1"/>
 <junction x="76.2" y="-8.89"/>
 <pinref part="D7" gate="G$1" pin="2"/>
@@
 <junction x="44.45" y="-30.48"/>
 <wire x1="48.26" y1="-30.48" x2="44.45" y2="-30.48" width="0.1524" layer="91"/>
-<pinref part="EC_UNBAL" gate="G$1" pin="1"/>
+<pinref part="EC_UB" gate="G$1" pin="1"/>
 <wire x1="48.26" y1="-30.48" x2="85.09" y2="-30.48" width="0.1524" layer="91"/>
 <junction x="48.26" y="-30.48"/>
@@
 <wire x1="81.28" y1="-22.86" x2="81.28" y2="-27.94" width="0.1524" layer="91"/>
 <junction x="81.28" y="-22.86"/>
-<pinref part="EN_UNBAL" gate="G$1" pin="1"/>
+<pinref part="EN_UB" gate="G$1" pin="1"/>
 <junction x="67.31" y="-27.94"/>
 <pinref part="D8" gate="G$1" pin="2"/>
@@
 <wire x1="63.5" y1="-17.78" x2="63.5" y2="-16.51" width="0.1524" layer="91"/>
 <junction x="63.5" y="-16.51"/>
-<pinref part="EN_UNBAL" gate="G$1" pin="2"/>
+<pinref part="EN_UB" gate="G$1" pin="2"/>
 <wire x1="67.31" y1="-17.78" x2="67.31" y2="-16.51" width="0.1524" layer="91"/>
 <wire x1="67.31" y1="-16.51" x2="63.5" y2="-16.51" width="0.1524" layer="91"/>
@@
 <wire x1="72.39" y1="3.81" x2="72.39" y2="6.35" width="0.1524" layer="91"/>
 <junction x="72.39" y="3.81"/>
-<pinref part="EP_UNBAL" gate="G$1" pin="2"/>
+<pinref part="EP_UB" gate="G$1" pin="2"/>
 <wire x1="76.2" y1="1.27" x2="76.2" y2="3.81" width="0.1524" layer="91"/>
 <wire x1="76.2" y1="3.81" x2="72.39" y2="3.81" width="0.1524" layer="91"/>
@@
 <pinref part="R3" gate="G$1" pin="1"/>
 <wire x1="44.45" y1="-19.05" x2="44.45" y2="-20.32" width="0.1524" layer="91"/>
-<pinref part="EC_UNBAL" gate="G$1" pin="2"/>
+<pinref part="EC_UB" gate="G$1" pin="2"/>
 <wire x1="48.26" y1="-20.32" x2="48.26" y2="-19.05" width="0.1524" layer="91"/>
 <wire x1="48.26" y1="-19.05" x2="44.45" y2="-19.05" width="0.1524" layer="91"/>
