File: Impedance_Potential_Board/Impedance_Potential.sch (EAGLE design)
At the start: 85 parts, among them IC1 MAX30001GCWV+, J1 Header, U4 AP2112K-1.8V

Commit message: Major Update
Parts:
- removed C24: 47nF, SparkFun-Capacitors:47NF-0603-25V-5%
- removed R3: 51k, SparkFun-Resistors:47KOHM-0603-1/10W-1%
- EC_UB: value JUMPER-SMT_2_NO_SILK -> JUMPER-SMT_2_NC_TRACE_SILK; device SparkFun-Jumpers:JUMPER-SMT_2_NO_SILK -> SparkFun-Jumpers:JUMPER-SMT_2_NC_TRACE_SILK
- R1, R2: value 51k -> 47k
- R18: device SparkFun-Resistors:100OHM-0603-1/4W-5% -> SparkFun-Resistors:100OHM-0603-1/10W-1%
- R19, R20, R21, R22: device SparkFun-Resistors:0OHM-0603-1/10W-5% -> SparkFun-Resistors:0OHM-0603-1/10W
- R23: value 0 -> 200k; device SparkFun-Resistors:0OHM-0603-1/10W-5% -> SparkFun-Resistors:200KOHM-0603-1/10W-1%
- R4: value 324k -> 330k
Connections:
- net ECGC: no longer C24.2, R3.2
- net N$2: no longer C24.1, R3.1
