File: Impedance_Potential_Board/Impedance_Potential.brd (EAGLE design)
At the start: 70 x 70 mm, 86 parts, among them IC1 MAX30001GCWV+, J1 Header, U4 AP2112K-1.8V

Commit message: Production Updates
Parts:
- removed EC_UNBAL, EN_UNBAL, EP_UNBAL: JUMPER-SMT_2_NO_SILK, SparkFun-Jumpers:SMT-JUMPER_2_NO_SILK
- added EC_UB, EN_UB, EP_UB: JUMPER-SMT_2_NO_SILK, SparkFun-Jumpers:SMT-JUMPER_2_NO_SILK
- U$1: device SparkFun-Aesthetics:OSHW-LOGO-M -> SparkFun-Aesthetics:OSHW-LOGO-S
- U4: device SparkFun-PowerIC:SOT23-5 -> AP2112K-1.8TRG1:SPARKFUN-POWERIC_SOT23-5
- moved P_UP_ENABLE 21.0 mm to (29.9, 64.5), turned to 0 degrees
- moved U$1 18.0 mm to (4.55, 16.9)
- moved C13 15.8 mm to (27.2, 31.8)
- moved C14 15.8 mm to (27.2, 33.3)
- moved U4 15.6 mm to (47.5, 30.9), turned to 180 degrees
- moved R22 15.3 mm to (16.8, 18.6)
- moved C15 14.4 mm to (44.0, 32.3), turned to 0 degrees
- moved EP_EN 13.9 mm to (20.4, 20.0)
- moved C16 13.7 mm to (49.2, 33.6), turned to 180 degrees
- moved C10 13.2 mm to (43.0, 28.4)
- moved AOUT 12.8 mm to (43.4, 30.8)
- moved R4 12.3 mm to (40.7, 24.7)
- moved C20 12.3 mm to (40.7, 22.2)
- moved R23 11.7 mm to (31.0, 18.6)
- moved C12 11.5 mm to (40.5, 33.1)
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Connections:
- net ECGC: now also EC_UB.1; no longer EC_UNBAL.1
- net ECGN: now also EN_UB.1; no longer EN_UNBAL.1
- net ECGP: now also EP_UB.1; no longer EP_UNBAL.1
- net N$1: now also EN_UB.2; no longer EN_UNBAL.2
- net N$2: now also EC_UB.2; no longer EC_UNBAL.2
- net N$3: now also EP_UB.2; no longer EP_UNBAL.2
Routing:
- net 3.3V: track 73.2 -> 107.6 mm, vias 2 -> 4
- net INTB_: track 21.6 -> 37.5 mm
- net INT2B_: track 19.9 -> 35.7 mm
- net SDO_: track 19.0 -> 34.5 mm
- net SDI_: track 18.2 -> 33.5 mm
- net N$1: track 20.2 -> 5.13 mm
- net SCLK_: track 17.6 -> 32.7 mm
- net CSB_: track 17.3 -> 32.1 mm
- net N$2: track 18.5 -> 5.18 mm, vias 2 -> 0
- net N$3: track 14.7 -> 5.13 mm
- net ECGN_: track 14.2 -> 22.5 mm
- net BIN: track 49.2 -> 41.5 mm, vias 3 -> 2
- net DRVP: track 29.4 -> 21.8 mm
- net GND: track 18.7 -> 12.0 mm, vias 105 -> 95
- net DRVN: track 29.4 -> 22.8 mm
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Other:
- board text added: "MAX Board MediBrick 2000"
- board text added: "Potential Impedance"
- board text removed: "MAX30001G Board MediBrick2000"

Commit message: Merging Production Status to Github, Obtaining senior design files
Routing:
- net 3.3V: track 107.6 -> 105.5 mm
- net GND: track 12.0 -> 11.5 mm
Other:
- board text added: "SCL"
- board text removed: "SCLK"
