File: Impedance_Potential_Board/Impedance_Potential.brd (EAGLE design)
At the start: 70 x 70 mm, 86 parts, among them IC1 MAX30001GCWV+, J1 Header, U4 AP2112K-1.8V

Commit message: Major Update
Parts:
- removed C24: 47nF, SparkFun-Capacitors:0603
- removed R3: 51k, SparkFun-Resistors:0603
- EC_UB: value JUMPER-SMT_2_NO_SILK -> JUMPER-SMT_2_NC_TRACE_SILK; device SparkFun-Jumpers:SMT-JUMPER_2_NO_SILK -> SparkFun-Jumpers:SMT-JUMPER_2_NC_TRACE_SILK
- R1, R2: value 51k -> 47k
- R23: value 0 -> 200k
- R4: value 324k -> 330k
- moved C20 11.6 mm to (29.8, 18.1), turned to 270 degrees
- moved R23 2.79 mm to (28.2, 18.1)
- moved ECGC 1.85 mm to (28.4, 15.2)
- moved R4 0.90 mm to (41.6, 24.7)
- moved BIP 0.83 mm to (31.6, 17.0)
- moved EC_UB 0.40 mm to (26.4, 16.9)
- moved C10 0.30 mm to (43.0, 28.1)
Connections:
- net ECGC: no longer C24.2, R3.2
- net N$2: no longer C24.1, R3.1
Routing:
- net ECGC: track 24.6 -> 21.1 mm
- net N$2: track 5.18 -> 1.97 mm
- net BIP: track 29.7 -> 31.5 mm
- net VCM: track 20.7 -> 22.0 mm, vias 4 -> 2
- net RBIAS: track 5.79 -> 6.39 mm
- net GND: vias 95 -> 94
