File: Thermistor_Board/using_MicroController_ADC/Temp.brd (EAGLE design)
At the start: 70 x 70 mm, 40 parts, among them J1 IO, J2 SJ-3523-SMT-TR, J3 SJ-3523-SMT-TR, J5 SJ-3523-SMT-TR

Commit message: Production Updates
Parts:
- moved U$1 3.20 mm to (5.70, 26.2)
Other:
- board text added: "Temperature Board MediBrick 2000"
- board text removed: "Temperature Board MediBrick2000"
