File: Stethoscope/with_integrated_ES8388/Sound.brd (EAGLE design)
At the start: 70 x 70 mm, 53 parts, among them IC1 ES8388, IC2 TLV9002IDDFR, J1 SJ-3523-SMT-TR, J3 SJ2-3574A-SMT-TR

Commit message: Production Updates
Connections:
- new net A_3.3V: C2.1, C3.1, IC2.8, J2.10, LS1.4, LS2.4, R16.2, R2.2
- net 3.3V: no longer C2.1, C3.1, IC2.8, LS1.4, LS2.4, R16.2, R2.2
Routing:
- net 3.3V: track 247.9 -> 140.6 mm, vias 5 -> 2
- net A_3.3V: track 0.00 -> 96.3 mm, vias 0 -> 2
- net GND: vias 76 -> 93
Other:
- board text removed: "NC"

Commit message: Sound Board Updates
Parts:
- added C28: 0.1uF, SparkFun-Capacitors:0603
- added C29: 10uF, SparkFun-Capacitors:0603
- added C30: 1nF, SparkFun-Capacitors:0603
- added J4: (no value), SparkFun-Connectors:1X02
- added R15, R17: 33, SparkFun-Resistors:0603
- added U1: MPRLS0300YG00001B, MPRLS0300YG00001B:MPRLS0300YG00001B
- R10, R11, R6, R7, R9: value 10k -> 33
- U$3: device SparkFun-Aesthetics:OSHW-LOGO-M -> SparkFun-Aesthetics:OSHW-LOGO-S
- moved U$3 6.32 mm to (5.45, 28.9)
- moved R11 0.60 mm to (14.1, 28.2)
Connections:
- new net EOC: J4.1, U1.8
- new net N$11: C30.2, U1.4
- new net N$6: R17.2, U1.2
- new net N$7: R15.2, U1.3
- new net N$9: C30.1, U1.6
- new net RST: J4.2, U1.9
- net 3.3V: now also C28.1, C29.1, U1.10
- net GND: now also C28.2, C29.2, U1.12
- net SCL: now also R15.1
- net SDA: now also R17.1
Routing:
- net 3.3V: track 140.6 -> 160.5 mm
- net SCL: track 49.7 -> 68.3 mm
- net SDA: track 49.1 -> 63.7 mm, vias 2 -> 3
- net EOC: track 0.00 -> 13.0 mm
- net RST: track 0.00 -> 7.53 mm
- net N$11: track 0.00 -> 2.54 mm
- net N$9: track 0.00 -> 2.45 mm
- net N$6: track 0.00 -> 2.38 mm
- net N$7: track 0.00 -> 2.35 mm
- net N$21: track 5.93 -> 5.33 mm
- net LRCLK: track 42.5 -> 42.0 mm
- net GND: vias 93 -> 98
Other:
- board text added: "EOC"
- board text added: "RST"
- board text added: "Sound & Pressure Board MediBrick2000"
- board text removed: "Sound Board MediBrick2000"
