File: IMU_Board/IMU.brd (EAGLE design)
At the start: 70 x 70 mm, 53 parts, among them J1 Header, Q1 BSS138, Q2 BSS138, Q3 BSS138, Q4 BSS138, Q5 BSS138, U1 ICM-20948, U3 BMP581, U4 AP2112K-1.8V

Commit message: Merging Production Status to Github, Obtaining senior design files
Parts:
- removed LED_EN: LED ENABLE, SparkFun-Jumpers:SMT-JUMPER_2_NC_PASTE_SILK
- removed PDWN_EN, PUP_EN: JUMPER-SMT_2_NC_PASTE_SILK, SparkFun-Jumpers:SMT-JUMPER_2_NC_PASTE_SILK
- added LED: LED ENABLE, SparkFun-Jumpers:SMT-JUMPER_2_NC_TRACE_SILK
- added PDWN, PUP: JUMPER-SMT_2_NC_PASTE_SILK, SparkFun-Jumpers:SMT-JUMPER_2_NC_PASTE_SILK
- moved U$1 2.93 mm to (3.05, 26.9)
- moved C1 1.50 mm to (50.1, 50.4)
- moved C13 1.50 mm to (58.1, 60.0)
- moved C14 1.50 mm to (58.1, 58.5)
- moved C15 1.50 mm to (58.9, 50.2)
- moved C16 1.50 mm to (58.0, 54.0)
- moved C17 1.50 mm to (52.1, 49.8)
- moved C2 1.50 mm to (42.2, 51.0)
- moved C21 1.50 mm to (53.6, 49.8)
- moved C3 1.50 mm to (48.2, 50.9)
- moved C4 1.50 mm to (37.5, 51.0)
- moved C5 1.50 mm to (39.0, 51.0)
- moved D1 1.50 mm to (60.7, 57.3)
- moved Q1 1.50 mm to (51.5, 56.2)
- moved Q2 1.50 mm to (48.1, 56.2)
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Connections:
- net 3.3V: now also PUP.1; no longer PUP_EN.1
- net GND: now also LED.1, PDWN.1; no longer LED_EN.1, PDWN_EN.1
- net N$28: now also LED.2; no longer LED_EN.2
- net N$29: now also PDWN.2; no longer PDWN_EN.2
- net N$30: now also PUP.2; no longer PUP_EN.2
Routing:
- net CS_581: track 6.20 -> 7.70 mm
- net SDI: track 6.22 -> 7.72 mm
- net SCL: track 6.41 -> 7.91 mm
- net INT_581: track 6.39 -> 7.89 mm
- net 3.3V: track 82.3 -> 83.8 mm
- net CS_20948: track 6.60 -> 8.10 mm
- net SDO: track 6.03 -> 7.53 mm
- net INT_20948: track 6.82 -> 8.32 mm
- net GND: vias 28 -> 31
Other:
- board text added: "CS2"
- board text added: "CS5"
- board text added: "INT2"
- board text added: "INT5"
- board text removed: "CS2X"
- board text removed: "CS5X"
- board text removed: "INT2X"
- board text removed: "INT5X"

Commit message: Passed Tests
Many sensors passed testing,
Many library updates
Parts:
- PUP: value JUMPER-SMT_2_NC_PASTE_SILK -> JUMPER-SMT_2_NC_TRACE_SILK; device SparkFun-Jumpers:SMT-JUMPER_2_NC_PASTE_SILK -> SparkFun-Jumpers:SMT-JUMPER_2_NC_TRACE_SILK
- R11, R12, R13, R15, R17, R24, R25: value 100k -> 10k
Changed lines of the file:
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@@
 <attribute name="VALUE" x="35.73" y="65.968" size="0.6096" layer="27" font="vector" ratio="20"/>
 </element>
-<element name="R11" library="SparkFun-Resistors" library_urn="urn:adsk.eagle:library:532" package="0603" package3d_urn="urn:adsk.eagle:package:41389018/1" value="100k" x="46.6" y="61.95" smashed="yes" rot="R270">
+<element name="R11" library="SparkFun-Resistors" library_urn="urn:adsk.eagle:library:532" package="0603" package3d_urn="urn:adsk.eagle:package:41389018/1" value="10k" x="46.6" y="61.95" smashed="yes" rot="R270">
 <attribute name="NAME" x="46.862" y="59.75" size="0.4064" layer="25" font="vector" ratio="10" rot="R270" align="bottom-center"/>
-<attribute name="PROD_ID" value="RES-07828" x="46.6" y="61.95" size="1.778" layer="27" rot="R270" display="off"/>
-<attribute name="VALUE" x="45.888" y="63.2" size="0.6096" layer="27" font="vector" ratio="20" rot="R270" align="top-center"/>
-</element>
-<element name="R12" library="SparkFun-Resistors" library_urn="urn:adsk.eagle:library:532" package="0603" package3d_urn="urn:adsk.eagle:package:41389018/1" value="100k" x="49.6" y="61.95" smashed="yes" rot="R270">
+<attribute name="PROD_ID" value="RES-00824" x="46.6" y="61.95" size="1.778" layer="27" rot="R270" display="off"/>
+<attribute name="VALUE" value="10k" x="45.888" y="63.2" size="0.6096" layer="27" font="vector" ratio="20" rot="R270" align="top-center"/>
+</element>
+<element name="R12" library="SparkFun-Resistors" library_urn="urn:adsk.eagle:library:532" package="0603" package3d_urn="urn:adsk.eagle:package:41389018/1" value="10k" x="49.6" y="61.95" smashed="yes" rot="R270">
 <attribute name="NAME" x="49.712" y="59.8" size="0.4064" layer="25" font="vector" ratio="10" rot="R270" align="bottom-center"/>
-<attribute name="PROD_ID" value="RES-07828" x="49.6" y="61.95" size="1.778" layer="27" rot="R270" display="off"/>
-<attribute name="VALUE" x="48.838" y="63.15" size="0.6096" layer="27" font="vector" ratio="20" rot="R270" align="top-center"/>
-</element>
-<element name="R13" library="SparkFun-Resistors" library_urn="urn:adsk.eagle:library:532" package="0603" package3d_urn="urn:adsk.eagle:package:41389018/1" value="100k" x="43.6" y="61.95" smashed="yes" rot="R270">
+<attribute name="PROD_ID" value="RES-00824" x="49.6" y="61.95" size="1.778" layer="27" rot="R270" display="off"/>
+<attribute name="VALUE" value="10k" x="48.838" y="63.15" size="0.6096" layer="27" font="vector" ratio="20" rot="R270" align="top-center"/>
+</element>
+<element name="R13" library="SparkFun-Resistors" library_urn="urn:adsk.eagle:library:532" package="0603" package3d_urn="urn:adsk.eagle:package:41389018/1" value="10k" x="43.6" y="61.95" smashed="yes" rot="R270">
 <attribute name="NAME" x="43.812" y="59.8" size="0.4064" layer="25" font="vector" ratio="10" rot="R270" align="bottom-center"/>
-<attribute name="PROD_ID" value="RES-07828" x="43.6" y="61.95" size="1.778" layer="27" rot="R270" display="off"/>
-<attribute name="VALUE" x="42.838" y="63.2" size="0.6096" layer="27" font="vector" ratio="20" rot="R270" align="top-center"/>
+<attribute name="PROD_ID" value="RES-00824" x="43.6" y="61.95" size="1.778" layer="27" rot="R270" display="off"/>
+<attribute name="VALUE" value="10k" x="42.838" y="63.2" size="0.6096" layer="27" font="vector" ratio="20" rot="R270" align="top-center"/>
 </element>
 <element name="PDWN" library="SparkFun-Jumpers" library_urn="urn:adsk.eagle:library:528" package="SMT-JUMPER_2_NC_PASTE_SILK" package3d_urn="urn:adsk.eagle:package:39282/1" value="JUMPER-SMT_2_NC_PASTE_SILK" x="59.0936" y="61.9" smashed="yes">
@@
 <attribute name="VALUE" x="59.0936" y="60.757" size="0.6096" layer="27" font="vector" ratio="20" align="top-center" display="off"/>
 </element>
-<element name="R15" library="SparkFun-Resistors" library_urn="urn:adsk.eagle:library:532" package="0603" package3d_urn="urn:adsk.eagle:package:41389018/1" value="100k" x="52.6" y="61.95" smashed="yes" rot="R270">
+<element name="R15" library="SparkFun-Resistors" library_urn="urn:adsk.eagle:library:532" package="0603" package3d_urn="urn:adsk.eagle:package:41389018/1" value="10k" x="52.6" y="61.95" smashed="yes" rot="R270">
 <attribute name="NAME" x="52.412" y="59.85" size="0.4064" layer="25" font="vector" ratio="10" rot="R270" align="bottom-center"/>
-<attribute name="PROD_ID" value="RES-07828" x="52.6" y="61.95" size="1.778" layer="27" rot="R270" display="off"/>
-<attribute name="VALUE" x="51.788" y="63.2" size="0.6096" layer="27" font="vector" ratio="20" rot="R270" align="top-center"/>
-</element>
-<element name="R17" library="SparkFun-Resistors" library_urn="urn:adsk.eagle:library:532" package="0603" package3d_urn="urn:adsk.eagle:package:41389018/1" value="100k" x="37.6" y="61.95" smashed="yes" rot="R270">
+<attribute name="PROD_ID" value="RES-00824" x="52.6" y="61.95" size="1.778" layer="27" rot="R270" display="off"/>
+<attribute name="VALUE" value="10k" x="51.788" y="63.2" size="0.6096" layer="27" font="vector" ratio="20" rot="R270" align="top-center"/>
+</element>
+<element name="R17" library="SparkFun-Resistors" library_urn="urn:adsk.eagle:library:532" package="0603" package3d_urn="urn:adsk.eagle:package:41389018/1" value="10k" x="37.6" y="61.95" smashed="yes" rot="R270">
 <attribute name="NAME" x="37.462" y="59.8" size="0.4064" layer="25" font="vector" ratio="10" rot="R270" align="bottom-center"/>
-<attribute name="PROD_ID" value="RES-07828" x="37.6" y="61.95" size="1.778" layer="27" rot="R270" display="off"/>
-<attribute name="VALUE" x="36.788" y="63.1" size="0.6096" layer="27" font="vector" ratio="20" rot="R270" align="top-center"/>
-</element>
-<element name="PUP" library="SparkFun-Jumpers" library_urn="urn:adsk.eagle:library:528" package="SMT-JUMPER_2_NC_PASTE_SILK" package3d_urn="urn:adsk.eagle:package:39282/1" value="JUMPER-SMT_2_NC_PASTE_SILK" x="59.0936" y="64" smashed="yes">
+<attribute name="PROD_ID" value="RES-00824" x="37.6" y="61.95" size="1.778" layer="27" rot="R270" display="off"/>
+<attribute name="VALUE" value="10k" x="36.788" y="63.1" size="0.6096" layer="27" font="vector" ratio="20" rot="R270" align="top-center"/>
+</element>
+<element name="PUP" library="SparkFun-Jumpers" library_urn="urn:adsk.eagle:library:528" package="SMT-JUMPER_2_NC_TRACE_SILK" package3d_urn="urn:adsk.eagle:package:39281/2" value="JUMPER-SMT_2_NC_TRACE_SILK" x="59.0936" y="64" smashed="yes">
 <attribute name="NAME" x="59.0936" y="65.343" size="0.8128" layer="25" font="vector" ratio="12" align="bottom-center"/>
 <attribute name="VALUE" x="59.0936" y="62.857" size="0.6096" layer="27" font="vector" ratio="20" align="top-center" display="off"/>
@@
 <attribute name="VALUE" x="53.338" y="61.95" size="0.6096" layer="27" font="vector" ratio="20" rot="R270" align="top-center"/>
 </element>
-<element name="R24" library="SparkFun-Resistors" library_urn="urn:adsk.eagle:library:532" package="0603" package3d_urn="urn:adsk.eagle:package:41389018/1" value="100k" x="40.6" y="61.95" smashed="yes" rot="R270">
+<element name="R24" library="SparkFun-Resistors" library_urn="urn:adsk.eagle:library:532" package="0603" package3d_urn="urn:adsk.eagle:package:41389018/1" value="10k" x="40.6" y="61.95" smashed="yes" rot="R270">
 <attribute name="NAME" x="40.462" y="59.85" size="0.4064" layer="25" font="vector" ratio="10" rot="R270" align="bottom-center"/>
-<attribute name="PROD_ID" value="RES-07828" x="40.6" y="61.95" size="1.778" layer="27" rot="R270" display="off"/>
-<attribute name="VALUE" x="39.838" y="61.95" size="0.6096" layer="27" font="vector" ratio="20" rot="R270" align="top-center"/>
-</element>
-<element name="R25" library="SparkFun-Resistors" library_urn="urn:adsk.eagle:library:532" package="0603" package3d_urn="urn:adsk.eagle:package:41389018/1" value="100k" x="55.6" y="61.95" smashed="yes" rot="R270">
+<attribute name="PROD_ID" value="RES-00824" x="40.6" y="61.95" size="1.778" layer="27" rot="R270" display="off"/>
+<attribute name="VALUE" value="10k" x="39.838" y="61.95" size="0.6096" layer="27" font="vector" ratio="20" rot="R270" align="top-center"/>
+</element>
+<element name="R25" library="SparkFun-Resistors" library_urn="urn:adsk.eagle:library:532" package="0603" package3d_urn="urn:adsk.eagle:package:41389018/1" value="10k" x="55.6" y="61.95" smashed="yes" rot="R270">
 <attribute name="NAME" x="55.512" y="59.8" size="0.4064" layer="25" font="vector" ratio="10" rot="R270" align="bottom-center"/>
-<attribute name="PROD_ID" value="RES-07828" x="55.6" y="61.95" size="1.778" layer="27" rot="R270" display="off"/>
-<attribute name="VALUE" x="54.838" y="61.95" size="0.6096" layer="27" font="vector" ratio="20" rot="R270" align="top-center"/>
+<attribute name="PROD_ID" value="RES-00824" x="55.6" y="61.95" size="1.778" layer="27" rot="R270" display="off"/>
+<attribute name="VALUE" value="10k" x="54.838" y="61.95" size="0.6096" layer="27" font="vector" ratio="20" rot="R270" align="top-center"/>
 </element>
 </elements>
@@
 <contactref element="R25" pad="1"/>
 <via x="60.45" y="63.95" extent="1-16" drill="0.35" diameter="0.75"/>
-<wire x1="59.5" y1="64" x2="60.35" y2="64" width="0.254" layer="1"/>
+<wire x1="59.6143" y1="64" x2="60.35" y2="64" width="0.254" layer="1"/>
 <wire x1="60.35" y1="64" x2="60.45" y2="63.95" width="0.254" layer="1"/>
 <via x="37.6" y="63.95" extent="1-16" drill="0.35" diameter="0.75"/>
@@
 <wire x1="57.2" y1="64.08" x2="54.78" y2="66.5" width="0.508" layer="1"/>
 <wire x1="57.2" y1="64.08" x2="57.2" y2="64" width="0.508" layer="1"/>
-<wire x1="58.6872" y1="64" x2="57.2" y2="64" width="0.254" layer="1"/>
+<wire x1="58.5729" y1="64" x2="57.2" y2="64" width="0.254" layer="1"/>
 <wire x1="57.2" y1="54.05" x2="57.2" y2="52.75" width="0.508" layer="1"/>
 <wire x1="57.2" y1="52.75" x2="57.2" y2="51.6501" width="0.508" layer="1"/>
