File: IMU_Board/IMU.sch (EAGLE design)
At the start: 52 parts, among them J1 Header, Q1 BSS138, Q2 BSS138, Q3 BSS138, Q4 BSS138, Q5 BSS138, U1 ICM-20948, U3 BMP581, U4 AP2112K-1.8V

Commit message: Merging Production Status to Github, Obtaining senior design files
Parts:
- removed LED_EN: LED ENABLE, SparkFun-Jumpers:JUMPER-SMT_2_NC_PASTE_SILK
- added LED: LED ENABLE, SparkFun-Jumpers:JUMPER-SMT_2_NC_TRACE_SILK
- renumbered PDWN_EN to PDWN, PUP_EN to PUP
Connections:
- net GND: now also LED.1; no longer LED_EN.1
- net N$28: now also LED.2; no longer LED_EN.2
Changed lines of the file:
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@@
 <part name="D1" library="SparkFun-LED" deviceset="LED-RED" device="0603" value="RED"/>
 <part name="GND4" library="SparkFun-Aesthetics" deviceset="GND" device=""/>
-<part name="LED_EN" library="SparkFun-Jumpers" library_urn="urn:adsk.eagle:library:528" deviceset="JUMPER-SMT_2_NC_PASTE" device="_SILK" package3d_urn="urn:adsk.eagle:package:39282/1" value="LED ENABLE"/>
+<part name="LED" library="SparkFun-Jumpers" library_urn="urn:adsk.eagle:library:528" deviceset="JUMPER-SMT_2_NC_TRACE" device="_SILK" package3d_urn="urn:adsk.eagle:package:39281/2" value="LED ENABLE"/>
 <part name="FRAME1" library="SparkFun-Aesthetics" library_urn="urn:adsk.eagle:library:507" deviceset="FRAME-LETTER" device="NO_PACKAGE" package3d_urn="urn:adsk.eagle:package:41384587/3"/>
 <part name="C15" library="SparkFun-Capacitors" deviceset="1.0UF" device="-0603-16V-10%" value="1.0uF"/>
@@
 <part name="R12" library="SparkFun-Resistors" library_urn="urn:adsk.eagle:library:532" deviceset="100KOHM" device="-0603-1/10W-1%" package3d_urn="urn:adsk.eagle:package:41389018/1" value="100k"/>
 <part name="R13" library="SparkFun-Resistors" library_urn="urn:adsk.eagle:library:532" deviceset="100KOHM" device="-0603-1/10W-1%" package3d_urn="urn:adsk.eagle:package:41389018/1" value="100k"/>
-<part name="PDWN_EN" library="SparkFun-Jumpers" library_urn="urn:adsk.eagle:library:528" deviceset="JUMPER-SMT_2_NC_PASTE" device="_SILK" package3d_urn="urn:adsk.eagle:package:39282/1" value="JUMPER-SMT_2_NC_PASTE_SILK"/>
+<part name="PDWN" library="SparkFun-Jumpers" library_urn="urn:adsk.eagle:library:528" deviceset="JUMPER-SMT_2_NC_PASTE" device="_SILK" package3d_urn="urn:adsk.eagle:package:39282/1" value="JUMPER-SMT_2_NC_PASTE_SILK"/>
 <part name="GND2" library="SparkFun-Aesthetics" deviceset="GND" device=""/>
 <part name="R15" library="SparkFun-Resistors" library_urn="urn:adsk.eagle:library:532" deviceset="100KOHM" device="-0603-1/10W-1%" package3d_urn="urn:adsk.eagle:package:41389018/1" value="100k"/>
 <part name="R17" library="SparkFun-Resistors" library_urn="urn:adsk.eagle:library:532" deviceset="100KOHM" device="-0603-1/10W-1%" package3d_urn="urn:adsk.eagle:package:41389018/1" value="100k"/>
-<part name="PUP_EN" library="SparkFun-Jumpers" library_urn="urn:adsk.eagle:library:528" deviceset="JUMPER-SMT_2_NC_PASTE" device="_SILK" package3d_urn="urn:adsk.eagle:package:39282/1" value="JUMPER-SMT_2_NC_PASTE_SILK"/>
+<part name="PUP" library="SparkFun-Jumpers" library_urn="urn:adsk.eagle:library:528" deviceset="JUMPER-SMT_2_NC_PASTE" device="_SILK" package3d_urn="urn:adsk.eagle:package:39282/1" value="JUMPER-SMT_2_NC_PASTE_SILK"/>
 <part name="C21" library="SparkFun-Capacitors" library_urn="urn:adsk.eagle:library:510" deviceset="10UF" device="-0603-6.3V-20%" package3d_urn="urn:adsk.eagle:package:41385090/1" value="10uF"/>
 <part name="GND3" library="supply1" deviceset="GND" device=""/>
@@
 <attribute name="VALUE" x="-33.02" y="-78.74" size="1.778" layer="96"/>
 </instance>
-<instance part="LED_EN" gate="G$1" x="-23.622" y="-71.12" smashed="yes">
+<instance part="LED" gate="G$1" x="-23.622" y="-71.12" smashed="yes">
 <attribute name="NAME" x="-26.162" y="-68.58" size="1.778" layer="95" font="vector"/>
 </instance>
@@
 <attribute name="VALUE" x="-109.982" y="-56.134" size="1.778" layer="96" font="vector" rot="R90" align="top-center"/>
 </instance>
-<instance part="PDWN_EN" gate="G$1" x="-101.6" y="-69.85" smashed="yes" rot="R90">
+<instance part="PDWN" gate="G$1" x="-101.6" y="-69.85" smashed="yes" rot="R90">
 <attribute name="NAME" x="-104.14" y="-80.01" size="1.778" layer="95" font="vector" rot="R90"/>
 </instance>
@@
 <attribute name="VALUE" x="-94.742" y="-56.134" size="1.778" layer="96" font="vector" rot="R90" align="top-center"/>
 </instance>
-<instance part="PUP_EN" gate="G$1" x="-86.36" y="-69.85" smashed="yes" rot="R90">
+<instance part="PUP" gate="G$1" x="-86.36" y="-69.85" smashed="yes" rot="R90">
 <attribute name="NAME" x="-88.9" y="-80.01" size="1.778" layer="95" font="vector" rot="R90"/>
 </instance>
@@
 <net name="GND" class="0">
 <segment>
-<pinref part="LED_EN" gate="G$1" pin="1"/>
+<pinref part="LED" gate="G$1" pin="1"/>
 <pinref part="GND4" gate="1" pin="GND"/>
 <wire x1="-30.48" y1="-73.66" x2="-30.48" y2="-71.12" width="0.1524" layer="91"/>
@@
 <segment>
 <pinref part="GND2" gate="1" pin="GND"/>
-<pinref part="PDWN_EN" gate="G$1" pin="1"/>
+<pinref part="PDWN" gate="G$1" pin="1"/>
 <wire x1="-101.6" y1="-76.2" x2="-101.6" y2="-74.93" width="0.1524" layer="91"/>
 </segment>
@@
 <segment>
 <pinref part="D1" gate="G$1" pin="C"/>
-<pinref part="LED_EN" gate="G$1" pin="2"/>
+<pinref part="LED" gate="G$1" pin="2"/>
 <wire x1="-8.382" y1="-71.12" x2="-18.542" y2="-71.12" width="0.1524" layer="91"/>
 </segment>
@@
 <wire x1="-96.52" y1="-62.23" x2="-96.52" y2="-60.96" width="0.1524" layer="91"/>
 <junction x="-101.6" y="-62.23"/>
-<pinref part="PDWN_EN" gate="G$1" pin="2"/>
+<pinref part="PDWN" gate="G$1" pin="2"/>
 <wire x1="-101.6" y1="-64.77" x2="-101.6" y2="-62.23" width="0.1524" layer="91"/>
 </segment>
@@
 <wire x1="-91.44" y1="-62.484" x2="-86.36" y2="-62.484" width="0.1524" layer="91"/>
 <junction x="-86.36" y="-62.484"/>
-<pinref part="PUP_EN" gate="G$1" pin="2"/>
+<pinref part="PUP" gate="G$1" pin="2"/>
 <wire x1="-86.36" y1="-64.77" x2="-86.36" y2="-62.484" width="0.1524" layer="91"/>
 <pinref part="R24" gate="G$1" pin="1"/>
@@
 </segment>
 <segment>
-<pinref part="PUP_EN" gate="G$1" pin="1"/>
+<pinref part="PUP" gate="G$1" pin="1"/>
 <wire x1="-86.36" y1="-74.93" x2="-86.36" y2="-76.2" width="0.1524" layer="91"/>
 <wire x1="-86.36" y1="-76.2" x2="-78.74" y2="-76.2" width="0.1524" layer="91"/>

Commit message: Passed Tests
Many sensors passed testing,
Many library updates
Parts:
- PUP: value JUMPER-SMT_2_NC_PASTE_SILK -> JUMPER-SMT_2_NC_TRACE_SILK; device SparkFun-Jumpers:JUMPER-SMT_2_NC_PASTE_SILK -> SparkFun-Jumpers:JUMPER-SMT_2_NC_TRACE_SILK
- R11, R12, R13, R15, R17, R24, R25: value 100k -> 10k; device SparkFun-Resistors:100KOHM-0603-1/10W-1% -> SparkFun-Resistors:10KOHM-0603-1/10W-1%
Other:
- note added: "Possible Improvements: - VDD in ICM can also go to 1.8V - FSYNC should be provided as input and pulled low - 10K resistors could be combined into chip with multiple resistor - level shifter should be combined into chip with 2 or more shifters (BSS138) - pull down at connector might not be needed. - pull up should be combined into chip with multiple resistors."
Changed lines of the file:
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@@
 <part name="J1" library="SparkFun-Connectors" library_urn="urn:adsk.eagle:library:513" deviceset="CONN_09" device="" package3d_urn="urn:adsk.eagle:package:38153/2" value="Header"/>
 <part name="GND1" library="supply1" deviceset="GND" device=""/>
-<part name="R11" library="SparkFun-Resistors" library_urn="urn:adsk.eagle:library:532" deviceset="100KOHM" device="-0603-1/10W-1%" package3d_urn="urn:adsk.eagle:package:41389018/1" value="100k"/>
-<part name="R12" library="SparkFun-Resistors" library_urn="urn:adsk.eagle:library:532" deviceset="100KOHM" device="-0603-1/10W-1%" package3d_urn="urn:adsk.eagle:package:41389018/1" value="100k"/>
-<part name="R13" library="SparkFun-Resistors" library_urn="urn:adsk.eagle:library:532" deviceset="100KOHM" device="-0603-1/10W-1%" package3d_urn="urn:adsk.eagle:package:41389018/1" value="100k"/>
+<part name="R11" library="SparkFun-Resistors" library_urn="urn:adsk.eagle:library:532" deviceset="10KOHM" device="-0603-1/10W-1%" package3d_urn="urn:adsk.eagle:package:41389018/1" value="10k"/>
+<part name="R12" library="SparkFun-Resistors" library_urn="urn:adsk.eagle:library:532" deviceset="10KOHM" device="-0603-1/10W-1%" package3d_urn="urn:adsk.eagle:package:41389018/1" value="10k"/>
+<part name="R13" library="SparkFun-Resistors" library_urn="urn:adsk.eagle:library:532" deviceset="10KOHM" device="-0603-1/10W-1%" package3d_urn="urn:adsk.eagle:package:41389018/1" value="10k"/>
 <part name="PDWN" library="SparkFun-Jumpers" library_urn="urn:adsk.eagle:library:528" deviceset="JUMPER-SMT_2_NC_PASTE" device="_SILK" package3d_urn="urn:adsk.eagle:package:39282/1" value="JUMPER-SMT_2_NC_PASTE_SILK"/>
 <part name="GND2" library="SparkFun-Aesthetics" deviceset="GND" device=""/>
-<part name="R15" library="SparkFun-Resistors" library_urn="urn:adsk.eagle:library:532" deviceset="100KOHM" device="-0603-1/10W-1%" package3d_urn="urn:adsk.eagle:package:41389018/1" value="100k"/>
-<part name="R17" library="SparkFun-Resistors" library_urn="urn:adsk.eagle:library:532" deviceset="100KOHM" device="-0603-1/10W-1%" package3d_urn="urn:adsk.eagle:package:41389018/1" value="100k"/>
-<part name="PUP" library="SparkFun-Jumpers" library_urn="urn:adsk.eagle:library:528" deviceset="JUMPER-SMT_2_NC_PASTE" device="_SILK" package3d_urn="urn:adsk.eagle:package:39282/1" value="JUMPER-SMT_2_NC_PASTE_SILK"/>
+<part name="R15" library="SparkFun-Resistors" library_urn="urn:adsk.eagle:library:532" deviceset="10KOHM" device="-0603-1/10W-1%" package3d_urn="urn:adsk.eagle:package:41389018/1" value="10k"/>
+<part name="R17" library="SparkFun-Resistors" library_urn="urn:adsk.eagle:library:532" deviceset="10KOHM" device="-0603-1/10W-1%" package3d_urn="urn:adsk.eagle:package:41389018/1" value="10k"/>
+<part name="PUP" library="SparkFun-Jumpers" library_urn="urn:adsk.eagle:library:528" deviceset="JUMPER-SMT_2_NC_TRACE" device="_SILK" package3d_urn="urn:adsk.eagle:package:39281/2" value="JUMPER-SMT_2_NC_TRACE_SILK"/>
 <part name="C21" library="SparkFun-Capacitors" library_urn="urn:adsk.eagle:library:510" deviceset="10UF" device="-0603-6.3V-20%" package3d_urn="urn:adsk.eagle:package:41385090/1" value="10uF"/>
 <part name="GND3" library="supply1" deviceset="GND" device=""/>
@@
 <part name="R28" library="SparkFun-Resistors" library_urn="urn:adsk.eagle:library:532" deviceset="10OHM" device="-0603-1/10W-1%" package3d_urn="urn:adsk.eagle:package:41389018/1" value="10"/>
 <part name="GND7" library="SparkFun-PowerSymbols" deviceset="GND" device=""/>
-<part name="R24" library="SparkFun-Resistors" library_urn="urn:adsk.eagle:library:532" deviceset="100KOHM" device="-0603-1/10W-1%" package3d_urn="urn:adsk.eagle:package:41389018/1" value="100k"/>
-<part name="R25" library="SparkFun-Resistors" library_urn="urn:adsk.eagle:library:532" deviceset="100KOHM" device="-0603-1/10W-1%" package3d_urn="urn:adsk.eagle:package:41389018/1" value="100k"/>
+<part name="R24" library="SparkFun-Resistors" library_urn="urn:adsk.eagle:library:532" deviceset="10KOHM" device="-0603-1/10W-1%" package3d_urn="urn:adsk.eagle:package:41389018/1" value="10k"/>
+<part name="R25" library="SparkFun-Resistors" library_urn="urn:adsk.eagle:library:532" deviceset="10KOHM" device="-0603-1/10W-1%" package3d_urn="urn:adsk.eagle:package:41389018/1" value="10k"/>
 </parts>
 <sheets>
@@
 <plain>
 <text x="43.18" y="-88.9" size="3.81" layer="91">Urs Utzinger</text>
+<text x="0" y="-43.18" size="1.778" layer="91">Possible Improvements:
+- VDD in ICM can also go to 1.8V
+- FSYNC should be provided as input and pulled low
+- 10K resistors could be combined into chip with multiple resistor
+- level shifter should be combined into chip with 2 or more shifters (BSS138)
+- pull down at connector might not be needed.
+- pull up should be combined into chip with multiple resistors.</text>
 </plain>
 <instances>
@@
 </drawing>
 <compatibility>
+<note version="6.3" minversion="6.2.2" severity="warning">
+Since Version 6.2.2 text objects can contain more than one line,
+which will not be processed correctly with this version.
+</note>
 <note version="8.2" severity="warning">
 Since Version 8.2, EAGLE supports online libraries. The ids
