File: Thermistor_Board/Temp.brd (EAGLE design)
At the start: 70 x 70 mm, 43 parts, among them J1 IO, J2 SJ-3523-SMT-TR, J3 SJ-3523-SMT-TR, J5 SJ-3523-SMT-TR

Commit message: Passed Tests
Many sensors passed testing,
Many library updates
Parts:
- R2, R3, R4, R6, R7, R9: value 10k -> 20k
